Commit message: WIP urdf of hand by Mathias

File: festo_phand_description/urdf/finger_macro.xacro (robot description, xacro)
@@ -1,5 +1,5 @@
 <?xml version="1.0"?>
-<robot name="bigfinger" xmlns:xacro="http://ros.org/wiki/xacro">
-    <xacro:macro name="bigfinger" params="prefix version">
+<robot name="finger" xmlns:xacro="http://ros.org/wiki/xacro">
+    <xacro:macro name="finger" params="prefix version">
         <link
                 name="${prefix}base_link">
@@ -75,7 +75,7 @@
                     rpy="1.5708 0 0"/>
             <parent
-                    link="base_link"/>
-            <child
-                    link="fake_intermediate_1"/>
+                    link="${prefix}base_link"/>
+            <child
+                    link="${prefix}fake_intermediate_1"/>
             <axis
                     xyz="0 1 0"/>
@@ -119,15 +119,15 @@
                     rpy="0 0 0"/>
             <parent
-                    link="fake_intermediate_1"/>
-            <child
-                    link="fake_intermediate_2"/>
-            <axis
-                    xyz="0 1 0"/>
-            <limit
-                    lower="0"
-                    upper="0.25"
-                    effort="0"
-                    velocity="0"/>
-            <mimic joint="joint_1"/>
+                    link="${prefix}fake_intermediate_1"/>
+            <child
+                    link="${prefix}fake_intermediate_2"/>
+            <axis
+                    xyz="0 1 0"/>
+            <limit
+                    lower="0"
+                    upper="0.25"
+                    effort="0"
+                    velocity="0"/>
+            <mimic joint="${prefix}joint_1"/>
         </joint>
         <link
@@ -178,15 +178,15 @@
                     rpy="0 0 0"/>
             <parent
-                    link="fake_intermediate_2"/>
-            <child
-                    link="fake_intermediate_3"/>
-            <axis
-                    xyz="0 1 0"/>
-            <limit
-                    lower="0"
-                    upper="0.25"
-                    effort="0"
-                    velocity="0"/>
-            <mimic joint="joint_1"/>
+                    link="${prefix}fake_intermediate_2"/>
+            <child
+                    link="${prefix}fake_intermediate_3"/>
+            <axis
+                    xyz="0 1 0"/>
+            <limit
+                    lower="0"
+                    upper="0.25"
+                    effort="0"
+                    velocity="0"/>
+            <mimic joint="${prefix}joint_1"/>
         </joint>
         <link
@@ -237,15 +237,15 @@
                     rpy="0 0 0"/>
             <parent
-                    link="fake_intermediate_3"/>
-            <child
-                    link="fake_intermediate_4"/>
-            <axis
-                    xyz="0 1 0"/>
-            <limit
-                    lower="0"
-                    upper="0.25"
-                    effort="0"
-                    velocity="0"/>
-            <mimic joint="joint_1"/>
+                    link="${prefix}fake_intermediate_3"/>
+            <child
+                    link="${prefix}fake_intermediate_4"/>
+            <axis
+                    xyz="0 1 0"/>
+            <limit
+                    lower="0"
+                    upper="0.25"
+                    effort="0"
+                    velocity="0"/>
+            <mimic joint="${prefix}joint_1"/>
         </joint>
         <link
@@ -286,15 +286,15 @@
                     rpy="0 0 0"/>
             <parent
-                    link="fake_intermediate_4"/>
-            <child
-                    link="Phallanx_1"/>
-            <axis
-                    xyz="0 1 0"/>
-            <limit
-                    lower="0"
-                    upper="0.25"
-                    effort="0"
-                    velocity="0"/>
-            <mimic joint="joint_1"/>
+                    link="${prefix}fake_intermediate_4"/>
+            <child
+                    link="${prefix}Phallanx_1"/>
+            <axis
+                    xyz="0 1 0"/>
+            <limit
+                    lower="0"
+                    upper="0.25"
+                    effort="0"
+                    velocity="0"/>
+            <mimic joint="${prefix}joint_1"/>
         </joint>
         <link
@@ -338,7 +338,7 @@
             </xacro:if>
             <parent
-                    link="Phallanx_1"/>
-            <child
-                    link="fake_intermediate_5"/>
+                    link="${prefix}Phallanx_1"/>
+            <child
+                    link="${prefix}fake_intermediate_5"/>
             <axis
                     xyz="0 1 0"/>
@@ -396,15 +396,15 @@
                     rpy="0 0 0"/>
             <parent
-                    link="fake_intermediate_5"/>
-            <child
-                    link="fake_intermediate_6"/>
-            <axis
-                    xyz="0 1 0"/>
-            <limit
-                    lower="0"
-                    upper="0.25"
-                    effort="0"
-                    velocity="0"/>
-            <mimic joint="joint_6"/>
+                    link="${prefix}fake_intermediate_5"/>
+            <child
+                    link="${prefix}fake_intermediate_6"/>
+            <axis
+                    xyz="0 1 0"/>
+            <limit
+                    lower="0"
+                    upper="0.25"
+                    effort="0"
+                    velocity="0"/>
+            <mimic joint="${prefix}joint_6"/>
         </joint>
         <link
@@ -455,15 +455,15 @@
                     rpy="0 0 0"/>
             <parent
-                    link="fake_intermediate_6"/>
-            <child
-                    link="fake_intermediate_7"/>
-            <axis
-                    xyz="0 1 0"/>
-            <limit
-                    lower="0"
-                    upper="0.25"
-                    effort="0"
-                    velocity="0"/>
-            <mimic joint="joint_6"/>
+                    link="${prefix}fake_intermediate_6"/>
+            <child
+                    link="${prefix}fake_intermediate_7"/>
+            <axis
+                    xyz="0 1 0"/>
+            <limit
+                    lower="0"
+                    upper="0.25"
+                    effort="0"
+                    velocity="0"/>
+            <mimic joint="${prefix}joint_6"/>
         </joint>
         <link
@@ -518,15 +518,15 @@
                     rpy="0 0 0"/>
             <parent
-                    link="fake_intermediate_7"/>
-            <child
-                    link="Phallanx_2"/>
-            <axis
-                    xyz="0 1 0"/>
-            <limit
-                    lower="0"
-                    upper="0.25"
-                    effort="0"
-                    velocity="0"/>
-            <mimic joint="joint_6"/>
+                    link="${prefix}fake_intermediate_7"/>
+            <child
+                    link="${prefix}Phallanx_2"/>
+            <axis
+                    xyz="0 1 0"/>
+            <limit
+                    lower="0"
+                    upper="0.25"
+                    effort="0"
+                    velocity="0"/>
+            <mimic joint="${prefix}joint_6"/>
         </joint>
         <link
@@ -584,15 +584,15 @@
             </xacro:if>
             <parent
-                    link="Phallanx_2"/>
-            <child
-                    link="fake_intermediate_8"/>
-            <axis
-                    xyz="0 1 0"/>
-            <limit
-                    lower="0"
-                    upper="0.25"
-                    effort="0"
-                    velocity="0"/>
-            <mimic joint="joint_6"/>
+                    link="${prefix}Phallanx_2"/>
+            <child
+                    link="${prefix}fake_intermediate_8"/>
+            <axis
+                    xyz="0 1 0"/>
+            <limit
+                    lower="0"
+                    upper="0.25"
+                    effort="0"
+                    velocity="0"/>
+            <mimic joint="${prefix}joint_6"/>
         </joint>
         <link
@@ -643,15 +643,15 @@
                     rpy="0 0 0"/>
             <parent
-                    link="fake_intermediate_8"/>
-            <child
-                    link="fake_intermediate_9"/>
-            <axis
-                    xyz="0 1 0"/>
-            <limit
-                    lower="0"
-                    upper="0.25"
-                    effort="0"
-                    velocity="0"/>
-            <mimic joint="joint_6"/>
+                    link="${prefix}fake_intermediate_8"/>
+            <child
+                    link="${prefix}fake_intermediate_9"/>
+            <axis
+                    xyz="0 1 0"/>
+            <limit
+                    lower="0"
+                    upper="0.25"
+                    effort="0"
+                    velocity="0"/>
+            <mimic joint="${prefix}joint_6"/>
         </joint>
         <link
@@ -702,15 +702,15 @@
                     rpy="0 0 0"/>
             <parent
-                    link="fake_intermediate_9"/>
-            <child
-                    link="fake_intermediate_10"/>
-            <axis
-                    xyz="0 1 0"/>
-            <limit
-                    lower="0"
-                    upper="0.25"
-                    effort="0"
-                    velocity="0"/>
-            <mimic joint="joint_6"/>
+                    link="${prefix}fake_intermediate_9"/>
+            <child
+                    link="${prefix}fake_intermediate_10"/>
+            <axis
+                    xyz="0 1 0"/>
+            <limit
+                    lower="0"
+                    upper="0.25"
+                    effort="0"
+                    velocity="0"/>
+            <mimic joint="${prefix}joint_6"/>
         </joint>
         <link
@@ -761,15 +761,15 @@
                     rpy="3.1416 0 3.1416"/>
             <parent
-                    link="fake_intermediate_10"/>
-            <child
-                    link="tip_link"/>
-            <axis
-                    xyz="0 1 0"/>
-            <limit
-                    lower="0"
-                    upper="0.25"
-                    effort="0"
-                    velocity="0"/>
-            <mimic joint="joint_6"/>
+                    link="${prefix}fake_intermediate_10"/>
+            <child
+                    link="${prefix}tip_link"/>
+            <axis
+                    xyz="0 1 0"/>
+            <limit
+                    lower="0"
+                    upper="0.25"
+                    effort="0"
+                    velocity="0"/>
+            <mimic joint="${prefix}joint_6"/>
         </joint>
     </xacro:macro>

Commit message: WIP hand urdf, angles cylinders from wrist now work

File: festo_phand_description/urdf/finger_macro.xacro (robot description, xacro)
@@ -26,9 +26,5 @@
                             filename="package://festo_phand_description/meshes/finger/base_link.STL"/>
                 </geometry>
-                <material
-                        name="${prefix}">
-                    <color
-                            rgba="0.792156862745098 0.819607843137255 0.933333333333333 1"/>
-                </material>
+<xacro:grey />
             </visual>
             <collision>
@@ -52,9 +48,5 @@
                             filename="package://festo_phand_description/meshes/finger/fake_intermediate.STL"/>
                 </geometry>
-                <material
-                        name="${prefix}">
-                    <color
-                            rgba="0.792156862745098 0.819607843137255 0.933333333333333 1"/>
-                </material>
+<xacro:grey />
             </visual>
             <collision>
@@ -96,9 +88,5 @@
                             filename="package://festo_phand_description/meshes/finger/fake_intermediate.STL"/>
                 </geometry>
-                <material
-                        name="${prefix}">
-                    <color
-                            rgba="0.792156862745098 0.819607843137255 0.933333333333333 1"/>
-                </material>
+<xacro:grey />
             </visual>
             <collision>
@@ -155,9 +143,5 @@
                             filename="package://festo_phand_description/meshes/finger/fake_intermediate.STL"/>
                 </geometry>
-                <material
-                        name="${prefix}">
-                    <color
-                            rgba="0.792156862745098 0.819607843137255 0.933333333333333 1"/>
-                </material>
+<xacro:grey />
             </visual>
             <collision>
@@ -214,9 +198,5 @@
                             filename="package://festo_phand_description/meshes/finger/fake_intermediate.STL"/>
                 </geometry>
-                <material
-                        name="${prefix}">
-                    <color
-                            rgba="0.792156862745098 0.819607843137255 0.933333333333333 1"/>
-                </material>
+<xacro:grey />
             </visual>
             <collision>
@@ -263,9 +243,5 @@
                     </xacro:if>
                 </geometry>
-                <material
-                        name="${prefix}">
-                    <color
-                            rgba="0.792156862745098 0.819607843137255 0.933333333333333 1"/>
-                </material>
+<xacro:grey />
             </visual>
             <collision>
@@ -308,9 +284,5 @@
                             filename="package://festo_phand_description/meshes/finger/fake_intermediate.STL"/>
                 </geometry>
-                <material
-                        name="${prefix}">
-                    <color
-                            rgba="0.792156862745098 0.819607843137255 0.933333333333333 1"/>
-                </material>
+<xacro:grey />
             </visual>
             <collision>
@@ -373,9 +345,5 @@
                             filename="package://festo_phand_description/meshes/finger/fake_intermediate.STL"/>
                 </geometry>
-                <material
-                        name="${prefix}">
-                    <color
-                            rgba="0.792156862745098 0.819607843137255 0.933333333333333 1"/>
-                </material>
+<xacro:grey />
             </visual>
             <collision>
@@ -432,9 +400,5 @@
                             filename="package://festo_phand_description/meshes/finger/fake_intermediate.STL"/>
                 </geometry>
-                <material
-                        name="${prefix}">
-                    <color
-                            rgba="0.792156862745098 0.819607843137255 0.933333333333333 1"/>
-                </material>
+<xacro:grey />
             </visual>
             <collision>
@@ -495,9 +459,5 @@
                     </xacro:if>
                 </geometry>
-                <material
-                        name="${prefix}">
-                    <color
-                            rgba="0.792156862745098 0.819607843137255 0.933333333333333 1"/>
-                </material>
+<xacro:grey />
             </visual>
             <collision>
@@ -554,9 +514,5 @@
                             filename="package://festo_phand_description/meshes/finger/fake_intermediate.STL"/>
                 </geometry>
-                <material
-                        name="${prefix}">
-                    <color
-                            rgba="0.792156862745098 0.819607843137255 0.933333333333333 1"/>
-                </material>
+<xacro:grey />
             </visual>
             <collision>
@@ -620,9 +576,5 @@
                             filename="package://festo_phand_description/meshes/finger/fake_intermediate.STL"/>
                 </geometry>
-                <material
-                        name="${prefix}">
-                    <color
-                            rgba="0.792156862745098 0.819607843137255 0.933333333333333 1"/>
-                </material>
+<xacro:grey />
             </visual>
             <collision>
@@ -679,9 +631,5 @@
                             filename="package://festo_phand_description/meshes/finger/fake_intermediate.STL"/>
                 </geometry>
-                <material
-                        name="${prefix}">
-                    <color
-                            rgba="0.792156862745098 0.819607843137255 0.933333333333333 1"/>
-                </material>
+<xacro:grey />
             </visual>
             <collision>
@@ -738,9 +686,5 @@
                             filename="package://festo_phand_description/meshes/finger/tip_link.STL"/>
                 </geometry>
-                <material
-                        name="${prefix}">
-                    <color
-                            rgba="0.792156862745098 0.819607843137255 0.933333333333333 1"/>
-                </material>
+<xacro:grey />
             </visual>
             <collision>

File: festo_phand_description/urdf/full_hand.xacro (robot description, xacro)
@@ -6,4 +6,5 @@
   <xacro:include filename="$(find festo_phand_description)/urdf/thumb_macro.xacro" />
   <xacro:include filename="$(find festo_phand_description)/urdf/hand_macro.xacro" />
+  <xacro:include filename="$(find festo_phand_description)/urdf/common_material_and_constants.xacro" />
     <xacro:wrist  prefix="" version="" />
     <xacro:finger  prefix="pinky_" version="small" />
@@ -173,5 +174,5 @@
             <origin
                     xyz="-0.02396 0.02209 0.03342"
-                    rpy="0.56 -0.141 1.15"/> //1.588 0.078 0
+                    rpy="0 -0.141 1.15"/> //1.588 0.078 0
             <parent link="hand"/>
             <child link="cylinder_base"/>

File: festo_phand_description/urdf/hand_macro.xacro (robot description, xacro)
@@ -11,9 +11,5 @@
                         <mesh filename="package://festo_phand_description/meshes/hand.STL"/>
                 </geometry>
-                <material
-                        name="${prefix}">
-                    <color
-                            rgba="0.792156862745098 0.819607843137255 0.933333333333333 1"/>
-                </material>
+                    <xacro:black />
             </visual>
             <collision>

File: festo_phand_description/urdf/wrist_macro.xacro (robot description, xacro)
@@ -11,9 +11,5 @@
                         <mesh filename="package://festo_phand_description/meshes/wrist/wrist_base.STL"/>
                 </geometry>
-                <material
-                        name="${prefix}">
-                    <color
-                            rgba="0.792156862745098 0.819607843137255 0.933333333333333 1"/>
-                </material>
+                     <xacro:black />
             </visual>
             <collision>
@@ -35,9 +31,5 @@
                     <mesh filename="package://festo_phand_description/meshes/wrist/wrist_top.STL"/>
                 </geometry>
-                <material
-                        name="${prefix}">
-                    <color
-                            rgba="0 0.819607843137255 0.933333333333333 1"/>
-                </material>
+                    <xacro:black />
             </visual>
             <collision>
