Commit message: added small debug gui, fixed urdf hand

File: festo_phand_description/urdf/finger_macro.xacro (robot description, xacro)
@@ -1,5 +1,5 @@
 <?xml version="1.0"?>
 <robot name="finger" xmlns:xacro="http://ros.org/wiki/xacro">
-    <xacro:macro name="finger" params="prefix version">
+    <xacro:macro name="finger" params="prefix version linkchambers">
         <link
                 name="${prefix}base_link">
@@ -309,4 +309,7 @@
                         rpy="0 0 0"/>
             </xacro:if>
+            <xacro:if value="${linkjoint6!=''}">
+                <mimic joint="${linkto}"/>
+            </xacro:if>
             <parent
                     link="${prefix}Phallanx_1"/>

File: festo_phand_description/urdf/full_hand.xacro (robot description, xacro)
@@ -1,4 +1,6 @@
 <?xml version="1.0"?>
-<robot name="full_hand" xmlns:xacro="http://ros.org/wiki/xacro">
+<robot name="phand" xmlns:xacro="http://ros.org/wiki/xacro">
+    <xacro:macro name="phand" params="prefix">
+  <xacro:include filename="$(find festo_phand_description)/urdf/common_material_and_constants.xacro" />
   <xacro:include filename="$(find festo_phand_description)/urdf/wrist_macro.xacro" />
   <xacro:include filename="$(find festo_phand_description)/urdf/finger_macro.xacro" />
@@ -6,53 +8,52 @@
   <xacro:include filename="$(find festo_phand_description)/urdf/thumb_macro.xacro" />
   <xacro:include filename="$(find festo_phand_description)/urdf/hand_macro.xacro" />
-  <xacro:include filename="$(find festo_phand_description)/urdf/common_material_and_constants.xacro" />
-    <xacro:wrist  prefix="" version="" />
-    <xacro:finger  prefix="pinky_" version="small" />
-    <xacro:finger  prefix="ring" version="big" />
-    <xacro:finger  prefix="middle" version="big" />
-    <xacro:finger  prefix="index" version="big" />
-    <xacro:thumb  prefix="" version="" />
-    <xacro:cylinder  prefix="" version="index" />
-    <xacro:cylinder  prefix="left" version="wrist" />
-    <xacro:cylinder  prefix="right" version="wrist" />
-    <xacro:hand  prefix="" version="" />
-   <link name="base_link" >
+    <xacro:wrist  prefix="${prefix}" version="" />
+    <xacro:finger  prefix="${prefix}pinky_" version="small" linkjoint6="${prefix}pinky_joint1" linkjoint1="" />
+    <xacro:finger  prefix="${prefix}ring" version="big" linkjoint6="" linkjoint1=""/>
+    <xacro:finger  prefix="${prefix}middle" version="big" linkjoint6="${prefix}ring_" linkjoint1=""/>
+    <xacro:finger  prefix="${prefix}index" version="big" linkjoint6="" linkjoint1=""/>
+    <xacro:thumb  prefix="${prefix}" version="" linkjoint6="" linkjoint1=""/>
+    <xacro:cylinder  prefix="${prefix}" version="index" />
+    <xacro:cylinder  prefix="${prefix}left" version="wrist" />
+    <xacro:cylinder  prefix="${prefix}right" version="wrist" />
+    <xacro:hand  prefix="${prefix}" version="" />
+   <link name="${prefix}eef_link" >
    </link>
     <joint
-           name="base_joint"
+           name="${prefix}base_joint"
         type="fixed">
             <origin
-                    xyz="0 0 0"
+                    xyz="0 0 0.22232"
                     rpy="0 0 0"/> //1.629 -0.248 -0.326
-            <parent link="base_link"/>
-            <child link="wrist_base"/>
+            <parent link="${prefix}eef_link"/>
+            <child link="${prefix}wrist_base"/>
     </joint>
     //pinky
-  <link name="pinky_base_dummy" >
-  </link>
-    <joint
-           name="hand_pinky"
+  <link name="${prefix}pinky_base_dummy" >
+  </link>
+    <joint
+           name="${prefix}hand_pinky"
                 type="fixed">
             <origin
                     xyz="-0.04879 0.01961  0.12328"
                     rpy="1.643 -0.319 0"/> //1.629 -0.248 -0.326 .643 -0.319 0
-            <parent link="hand"/>
-            <child link="pinky_base_dummy"/>
-            <axis
-                    xyz="0 0 0"/>
-                <limit
-                    lower="0"
-                    upper="0"
-                    effort="0"
-                    velocity="0"/>
-  </joint>
-    <joint
-           name="hand_pinky2"
+            <parent link="${prefix}hand"/>
+            <child link="${prefix}pinky_base_dummy"/>
+            <axis
+                    xyz="0 0 0"/>
+                <limit
+                    lower="0"
+                    upper="0"
+                    effort="0"
+                    velocity="0"/>
+  </joint>
+    <joint
+           name="${prefix}hand_pinky2"
                 type="fixed">
             <origin
                     xyz="0 0 0"
                     rpy=" 0 1.57 0"/> //1.629 -0.248 -0.326
-            <parent link="pinky_base_dummy"/>
-            <child link="pinky_base_link"/>
+            <parent link="${prefix}pinky_base_dummy"/>
+            <child link="${prefix}pinky_base_link"/>
             <axis
                     xyz="0 0 0"/>
@@ -64,30 +65,30 @@
   </joint>
     //ring
-  <link name="ring_base_dummy" >
-  </link>
-    <joint
-           name="hand_ring"
+  <link name="${prefix}ring_base_dummy" >
+  </link>
+    <joint
+           name="${prefix}hand_ring"
                 type="fixed">
             <origin
                     xyz="-0.0182 0.02676 0.13027"
                     rpy="1.49 -0.055 0"/> //1.629 -0.248 -0.326
-            <parent link="hand"/>
-            <child link="ring_base_dummy"/>
-            <axis
-                    xyz="0 0 0"/>
-                <limit
-                    lower="0"
-                    upper="0"
-                    effort="0"
-                    velocity="0"/>
-    </joint>
-    <joint
-           name="hand_ring2"
+            <parent link="${prefix}hand"/>
+            <child link="${prefix}ring_base_dummy"/>
+            <axis
+                    xyz="0 0 0"/>
+                <limit
+                    lower="0"
+                    upper="0"
+                    effort="0"
+                    velocity="0"/>
+    </joint>
+    <joint
+           name="${prefix}hand_ring2"
                 type="fixed">
             <origin
                     xyz="0 0 0"
                     rpy=" 0 1.57 0"/> //1.629 -0.248 -0.326
-            <parent link="ring_base_dummy"/>
-            <child link="ringbase_link"/>
+            <parent link="${prefix}ring_base_dummy"/>
+            <child link="${prefix}ringbase_link"/>
             <axis
                     xyz="0 0 0"/>
@@ -99,30 +100,30 @@
   </joint>
     //middle
-  <link name="middle_base_dummy" >
-  </link>
-    <joint
-           name="hand_middle"
+  <link name="${prefix}middle_base_dummy" >
+  </link>
+    <joint
+           name="${prefix}hand_middle"
                 type="fixed">
             <origin
                     xyz="0.00579 0.01641 0.13459"
                     rpy="1.588 0.078 0"/> //1.629 -0.248 -0.326
-            <parent link="hand"/>
-            <child link="middle_base_dummy"/>
-            <axis
-                    xyz="0 0 0"/>
-                <limit
-                    lower="0"
-                    upper="0"
-                    effort="0"
-                    velocity="0"/>
-    </joint>
-    <joint
-           name="middle_ring2"
+            <parent link="${prefix}hand"/>
+            <child link="${prefix}middle_base_dummy"/>
+            <axis
+                    xyz="0 0 0"/>
+                <limit
+                    lower="0"
+                    upper="0"
+                    effort="0"
+                    velocity="0"/>
+    </joint>
+    <joint
+           name="${prefix}middle_ring2"
                 type="fixed">
             <origin
                     xyz="0 0 0"
                     rpy=" 0 1.1 0"/> //1.629 -0.248 -0.326
-            <parent link="middle_base_dummy"/>
-            <child link="middlebase_link"/>
+            <parent link="${prefix}middle_base_dummy"/>
+            <child link="${prefix}middlebase_link"/>
             <axis
                     xyz="0 0 0"/>
@@ -134,30 +135,30 @@
   </joint>
     //index
-  <link name="index_base_dummy" >
-  </link>
-    <joint
-           name="indexBase_index"
+  <link name="${prefix}index_base_dummy" >
+  </link>
+    <joint
+           name="${prefix}indexBase_index"
                 type="fixed">
             <origin
                     xyz="0.0005 0.00634 0.03501"
                     rpy="1.588 0 0"/> //1.588 0.078 0
-            <parent link="index_base_joint"/>
-            <child link="index_base_dummy"/>
-            <axis
-                    xyz="0 0 0"/>
-                <limit
-                    lower="0"
-                    upper="0"
-                    effort="0"
-                    velocity="0"/>
-    </joint>
-    <joint
-           name="indexBase_index2"
+            <parent link="${prefix}index_base_joint"/>
+            <child link="${prefix}index_base_dummy"/>
+            <axis
+                    xyz="0 0 0"/>
+                <limit
+                    lower="0"
+                    upper="0"
+                    effort="0"
+                    velocity="0"/>
+    </joint>
+    <joint
+           name="${prefix}indexBase_index2"
                 type="fixed">
             <origin
                     xyz="0 0 0"
                     rpy=" 0 -0.4 0"/> //0 1.1 0
-            <parent link="index_base_dummy"/>
-            <child link="indexbase_link"/>
+            <parent link="${prefix}index_base_dummy"/>
+            <child link="${prefix}indexbase_link"/>
             <axis
                     xyz="0 0 0"/>
@@ -170,11 +171,11 @@
     //index_cylinder
     <joint
-           name="index_cylinder_base"
+           name="${prefix}index_cylinder_base"
                 type="revolute">
             <origin
                     xyz="-0.02396 0.02209 0.03342"
                     rpy="${(45)*M_PI/180} -0.141 1.15"/> //1.588 0.078 0
-            <parent link="hand"/>
-            <child link="cylinder_base"/>
+            <parent link="${prefix}hand"/>
+            <child link="${prefix}cylinder_base"/>
             <axis
                     xyz="-1 0 0"/>
@@ -185,29 +186,29 @@
                     velocity="0"/>
     </joint>
-    <joint
-           name="index_cylinder_tip"
-                type="revolute">
-            <origin
-                    xyz="0 0 0.04475"
-                    rpy="0 0 0"/> //1.588 0.078 0
-            <parent link="rod"/>
-            <child link="index_base_joint"/>
-            <axis
-                    xyz="0 0 0"/>
-                <limit
-                    lower="0"
-                    upper="0"
-                    effort="0"
-                    velocity="0"/>
-    </joint>
+<!--    <joint-->
+<!--           name="${prefix}index_cylinder_tip"-->
+<!--                type="revolute">-->
+<!--            <origin-->
+<!--                    xyz="0 0 0.04475"-->
+<!--                    rpy="0 0 0"/> //1.588 0.078 0-->
+<!--            <parent link="${prefix}rod"/>-->
+<!--            <child link="${prefix}index_base_joint"/>-->
+<!--            <axis-->
+<!--                    xyz="0 0 0"/>-->
+<!--                <limit-->
+<!--                    lower="0"-->
+<!--                    upper="1.0"-->
+<!--                    effort="0"-->
+<!--                    velocity="0"/>-->
+<!--    </joint>-->
     //thumb
     <joint
-           name="hand_thumb"
+           name="${prefix}hand_thumb"
                 type="fixed">
             <origin
                     xyz="0 0 0.025"
                     rpy="0 0 0"/> //1.588 0.078 0
-            <parent link="hand"/>
-            <child link="drive"/>
+            <parent link="${prefix}hand"/>
+            <child link="${prefix}drive"/>
             <axis
                     xyz="0 0 0"/>
@@ -225,11 +226,11 @@
 <!--  </link>-->
     <joint
-           name="hand_wrist"
+           name="${prefix}hand_wrist"
                 type="fixed">
             <origin
                     xyz="0.00489 -0.0341 0.02622"
                     rpy="-0.1682 -0.0842 -1.1466"/> //-0.145 -0.13 -1.15
-            <parent link="wrist_top"/>
-            <child link="hand"/>
+            <parent link="${prefix}wrist_top"/>
+            <child link="${prefix}hand"/>
             <axis
                     xyz="0 0 0"/>
@@ -275,16 +276,16 @@
     //forearm_cylinders
     //LEFT
-    <link name="horizontal_dummyL" >
-  </link>
-    <link name="vertical_dummyL" >
-  </link>
-    <joint
-           name="wristBase_horizontal_L"
+    <link name="${prefix}horizontal_dummyL" >
+  </link>
+    <link name="${prefix}vertical_dummyL" >
+  </link>
+    <joint
+           name="${prefix}wristBase_horizontal_L"
                 type="revolute">
             <origin
                     xyz="0.02702 0.02695 -0.15803"
                     rpy="0 0 0.349"/> //
-            <parent link="wrist_base"/>
-            <child link="horizontal_dummyL"/> //leftcylinder_base
+            <parent link="${prefix}wrist_base"/>
+            <child link="${prefix}horizontal_dummyL"/> //leftcylinder_base
             <axis
                     xyz="1 0 0"/>
@@ -296,11 +297,11 @@
     </joint>
     <joint
-           name="horizontal_L_vertical_L"
+           name="${prefix}horizontal_L_vertical_L"
                 type="revolute">
             <origin
                     xyz="-0.00928 0 0"
                     rpy="0 0 0"/> //
-            <parent link="horizontal_dummyL"/>
-            <child link="vertical_dummyL"/> //leftcylinder_base
+            <parent link="${prefix}horizontal_dummyL"/>
+            <child link="${prefix}vertical_dummyL"/> //leftcylinder_base
             <axis
                     xyz="0 1 0"/>
@@ -312,31 +313,31 @@
     </joint>
     <joint
-           name="vertical_L_leftcylinder_base"
+           name="${prefix}vertical_L_leftcylinder_base"
                 type="fixed">
             <origin
                     xyz="0.00928 0 0"
                     rpy="0 0 0"/> //
-            <parent link="vertical_dummyL"/>
-            <child link="leftcylinder_base"/> //
-            <axis
-                    xyz="0 0 0"/>
-                <limit
-                    lower="0"
-                    upper="0"
-                    effort="0"
-                    velocity="0"/>
-    </joint>
-    <link name="horizontal_dummyR" >
-  </link>
-    <link name="vertical_dummyR" >
-  </link>
-    <joint
-           name="wristBase_cylinderR"
+            <parent link="${prefix}vertical_dummyL"/>
+            <child link="${prefix}leftcylinder_base"/> //
+            <axis
+                    xyz="0 0 0"/>
+                <limit
+                    lower="0"
+                    upper="0"
+                    effort="0"
+                    velocity="0"/>
+    </joint>
+    <link name="${prefix}horizontal_dummyR" >
+  </link>
+    <link name="${prefix}vertical_dummyR" >
+  </link>
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
File: festo_phand_description/urdf/wrist_macro.xacro (robot description, xacro)
@@ -2,4 +2,18 @@
 <robot name="wrist" xmlns:xacro="http://ros.org/wiki/xacro">
     <xacro:macro name="wrist" params="prefix version">
+<!--        <link-->
+<!--                name="${prefix}eef_link">-->
+<!--        </link>-->
+<!--        <joint-->
+<!--                name="eef_link_joint"-->
+<!--                type="fixed">-->
+<!--            <origin-->
+<!--                    xyz="0 0 -0.22232"-->
+<!--                    rpy="0 0 0"/>-->
+<!--            <parent link="${prefix}wrist_base"/>-->
+<!--            <child link="${prefix}eef_link"/>-->
+<!--            <axis-->
+<!--                    xyz="1 0 0"/>-->
+<!--        </joint>-->
         <link
                 name="${prefix}wrist_base">
@@ -10,4 +24,24 @@
                 <geometry>
                         <mesh filename="package://festo_phand_description/meshes/wrist/wrist_base.STL"/>
+                </geometry>
+                     <xacro:black />
+            </visual>
+            <collision>
+                <origin
+                        xyz="0 0 0"
+                        rpy="0 0 0"/>
+                <geometry>
+                     <mesh filename="package://festo_phand_description/meshes/wrist/wrist_base.STL"/>
+                </geometry>
+            </collision>
+        </link>
+                <link
+                name="${prefix}wrist_base2">
+            <visual>
+                <origin
+                        xyz="0 0 0"
+                        rpy="0 0 0"/>
+                <geometry>
+                        <mesh filename="package://festo_phand_description/meshes/static_components.STL"/>
                 </geometry>
                      <xacro:black />
@@ -46,5 +80,5 @@
         </link>
         <joint
-                name="rotation_x"
+                name="${prefix}rotation_x"
                 type="revolute">
             <origin
@@ -61,6 +95,17 @@
                     velocity="4"/>
         </joint>
+        <joint
+                name="${prefix}base_covers"
+                type="fixed">
+            <origin
+                    xyz="0 0 0"
+                    rpy="0 0 0"/>
+            <parent link="${prefix}wrist_base"/>
+            <child link="${prefix}wrist_base2"/>
+            <axis
+                    xyz="1 0 0"/>
+        </joint>
          <joint
-                name="rotation_y"
+                name="${prefix}rotation_y"
                 type="revolute">
             <origin
