Commit message: WIP urdf + joint publischer

File: festo_phand_description/urdf/cylinder_macro.xacro (robot description, xacro)
@@ -101,7 +101,4 @@
                 name="${prefix}cylinder_rod"
                 type="prismatic">
-            <origin
-                    xyz="0 0 0"
-                    rpy="0 0 0"/>
             <parent link="${prefix}cylinder_base"/>
             <child link="${prefix}rod"/>
@@ -109,14 +106,20 @@
                     xyz="0 0 1"/>
             <xacro:if value="${version=='wrist'}">
+                <origin
+                    xyz="0 0 0.052"
+                    rpy="0 0 0"/>
                 <limit
-                    lower="0.037"
-                    upper="0.085"
+                    lower="-0.00"
+                    upper="0.037"
                     effort="0"
                     velocity="4"/>
             </xacro:if>
             <xacro:if value="${version=='index'}">
+                <origin
+                    xyz="0 0 0.0228"
+                    rpy="0 0 0"/>
                 <limit
-                    lower="0.015"
-                    upper="0.035"
+                    lower="0.02"
+                    upper="0.03"
                     effort="0"
                     velocity="4"/>

File: festo_phand_description/urdf/full_hand.xacro (robot description, xacro)
@@ -173,5 +173,5 @@
             <origin
                     xyz="-0.02396 0.02209 0.03342"
-                    rpy="0 -0.141 1.15"/> //1.588 0.078 0
+                    rpy="0.56 -0.141 1.15"/> //1.588 0.078 0
             <parent link="hand"/>
             <child link="cylinder_base"/>

File: festo_phand_description/urdf/hand_macro.xacro (robot description, xacro)
@@ -55,5 +55,5 @@
             <origin
                     xyz="0.02385 -0.00408 0.08704"
-                    rpy="0 -0.131 1.15"/> //0 -0.131 1.57
+                    rpy="0.09 -0.131 1.15"/> //0 -0.131 1.57
             <parent link="${prefix}hand"/>
             <child link="${prefix}index_base_joint"/>

Commit message: WIP hand urdf, finger deviation works with a offset

File: festo_phand_description/urdf/cylinder_macro.xacro (robot description, xacro)
@@ -39,7 +39,14 @@
                 name="${prefix}rod">
             <visual>
+                 <xacro:if value="${version=='wrist'}">
                 <origin
                         xyz="0 0 0"
                         rpy="0 0 0"/>
+                  </xacro:if>
+                <xacro:if value="${version=='index'}">
+                <origin
+                        xyz="0 0 0.0168"
+                        rpy="0 0 0"/>
+                  </xacro:if>
                 <geometry>
                     <xacro:if value="${version=='wrist'}">
@@ -117,9 +124,9 @@
             <xacro:if value="${version=='index'}">
                 <origin
-                    xyz="0 0 0.0228"
+                    xyz="0 0 0.00"
                     rpy="0 0 0"/>
                 <limit
-                    lower="0.02"
-                    upper="0.03"
+                    lower="0.01"
+                    upper="0.02"
                     effort="0"
                     velocity="4"/>

File: festo_phand_description/urdf/full_hand.xacro (robot description, xacro)
@@ -174,12 +174,12 @@
             <origin
                     xyz="-0.02396 0.02209 0.03342"
-                    rpy="0 -0.141 1.15"/> //1.588 0.078 0
+                    rpy="${(45)*M_PI/180} -0.141 1.15"/> //1.588 0.078 0
             <parent link="hand"/>
             <child link="cylinder_base"/>
             <axis
-                    xyz="1 0 0"/>
-                <limit
-                    lower="-1"
-                    upper="1"
+                    xyz="-1 0 0"/>
+                <limit
+                    lower="-3"
+                    upper="3"
                     effort="0"
                     velocity="0"/>

File: festo_phand_description/urdf/hand_macro.xacro (robot description, xacro)
@@ -51,5 +51,5 @@
             <origin
                     xyz="0.02385 -0.00408 0.08704"
-                    rpy="0.09 -0.131 1.15"/> //0 -0.131 1.57
+                    rpy="${(45-6)*M_PI/-180} -0.131 1.15"/> //0 -0.131 1.57
             <parent link="${prefix}hand"/>
             <child link="${prefix}index_base_joint"/>
@@ -57,6 +57,6 @@
                     xyz="1 0 0"/>
                 <limit
-                    lower="-1"
-                    upper="1"
+                    lower="-2"
+                    upper="2"
                     effort="0"
                     velocity="4"/>

Commit message: Generated convex hulls as collision meshes for the hand

File: festo_phand_description/urdf/cylinder_macro.xacro (robot description, xacro)
@@ -28,8 +28,8 @@
                 <geometry>
                      <xacro:if value="${version=='wrist'}">
-                        <mesh filename="package://festo_phand_description/meshes/cylinder/cylinder_base.STL"/>
+                        <mesh filename="package://festo_phand_description/meshes/cylinder/cylinder_base_convex.STL"/>
                     </xacro:if>
                     <xacro:if value="${version=='index'}">
-                        <mesh filename="package://festo_phand_description/meshes/cylinder/index_cylinder_base.STL"/>
+                        <mesh filename="package://festo_phand_description/meshes/cylinder/index_cylinder_base_convex.STL"/>
                     </xacro:if>
                 </geometry>
@@ -69,8 +69,8 @@
                 <geometry>
                     <xacro:if value="${version=='wrist'}">
-                        <mesh filename="package://festo_phand_description/meshes/cylinder/rod.STL"/>
+                        <mesh filename="package://festo_phand_description/meshes/cylinder/rod_convex.STL"/>
                     </xacro:if>
                     <xacro:if value="${version=='index'}">
-                        <mesh filename="package://festo_phand_description/meshes/cylinder/index_rod.STL"/>
+                        <mesh filename="package://festo_phand_description/meshes/cylinder/index_rod_convex.STL"/>
                     </xacro:if>
                 </geometry>
@@ -100,5 +100,5 @@
                     <geometry>
                         <mesh
-                                filename="package://festo_phand_description/meshes/cylinder/ball.STL"/>
+                                filename="package://festo_phand_description/meshes/cylinder/ball_convex.STL"/>
                     </geometry>
                 </collision>

File: festo_phand_description/urdf/finger_macro.xacro (robot description, xacro)
@@ -34,5 +34,5 @@
                 <geometry>
                     <mesh
-                            filename="package://festo_phand_description/meshes/finger/base_link.STL"/>
+                            filename="package://festo_phand_description/meshes/finger/base_link_convex.STL"/>
                 </geometry>
             </collision>
@@ -56,5 +56,5 @@
                 <geometry>
                     <mesh
-                            filename="package://festo_phand_description/meshes/finger/fake_intermediate.STL"/>
+                            filename="package://festo_phand_description/meshes/finger/fake_intermediate_convex.STL"/>
                 </geometry>
             </collision>
@@ -99,5 +99,5 @@
                 <geometry>
                     <mesh
-                            filename="package://festo_phand_description/meshes/finger/fake_intermediate.STL"/>
+                            filename="package://festo_phand_description/meshes/finger/fake_intermediate_convex.STL"/>
                 </geometry>
             </collision>
@@ -154,5 +154,5 @@
                 <geometry>
                     <mesh
-                            filename="package://festo_phand_description/meshes/finger/fake_intermediate.STL"/>
+                            filename="package://festo_phand_description/meshes/finger/fake_intermediate_convex.STL"/>
                 </geometry>
             </collision>
@@ -209,5 +209,5 @@
                 <geometry>
                     <mesh
-                            filename="package://festo_phand_description/meshes/finger/fake_intermediate.STL"/>
+                            filename="package://festo_phand_description/meshes/finger/fake_intermediate_convex.STL"/>
                 </geometry>
             </collision>
@@ -254,5 +254,5 @@
                 <geometry>
                     <mesh
-                            filename="package://festo_phand_description/meshes/finger/phallanx_big.STL"/>
+                            filename="package://festo_phand_description/meshes/finger/phallanx_big_convex.STL"/>
                 </geometry>
             </collision>
@@ -295,5 +295,5 @@
                 <geometry>
                     <mesh
-                            filename="package://festo_phand_description/meshes/finger/fake_intermediate.STL"/>
+                            filename="package://festo_phand_description/meshes/finger/fake_intermediate_convex.STL"/>
                 </geometry>
             </collision>
@@ -359,5 +359,5 @@
                 <geometry>
                     <mesh
-                            filename="package://festo_phand_description/meshes/finger/fake_intermediate.STL"/>
+                            filename="package://festo_phand_description/meshes/finger/fake_intermediate_convex.STL"/>
                 </geometry>
             </collision>
@@ -414,5 +414,5 @@
                 <geometry>
                     <mesh
-                            filename="package://festo_phand_description/meshes/finger/fake_intermediate.STL"/>
+                            filename="package://festo_phand_description/meshes/finger/fake_intermediate_convex.STL"/>
                 </geometry>
             </collision>
@@ -473,5 +473,5 @@
                 <geometry>
                     <mesh
-                            filename="package://festo_phand_description/meshes/finger/phallanx_small.STL"/>
+                            filename="package://festo_phand_description/meshes/finger/phallanx_small_convex.STL"/>
                 </geometry>
             </collision>
@@ -528,5 +528,5 @@
                 <geometry>
                     <mesh
-                            filename="package://festo_phand_description/meshes/finger/fake_intermediate.STL"/>
+                            filename="package://festo_phand_description/meshes/finger/fake_intermediate_convex.STL"/>
                 </geometry>
             </collision>
@@ -590,5 +590,5 @@
                 <geometry>
                     <mesh
-                            filename="package://festo_phand_description/meshes/finger/fake_intermediate.STL"/>
+                            filename="package://festo_phand_description/meshes/finger/fake_intermediate_convex.STL"/>
                 </geometry>
             </collision>
@@ -645,5 +645,5 @@
                 <geometry>
                     <mesh
-                            filename="package://festo_phand_description/meshes/finger/fake_intermediate.STL"/>
+                            filename="package://festo_phand_description/meshes/finger/fake_intermediate_convex.STL"/>
                 </geometry>
             </collision>
@@ -700,5 +700,5 @@
                 <geometry>
                     <mesh
-                            filename="package://festo_phand_description/meshes/finger/tip_link.STL"/>
+                            filename="package://festo_phand_description/meshes/finger/tip_link_convex.STL"/>
                 </geometry>
             </collision>

File: festo_phand_description/urdf/hand_macro.xacro (robot description, xacro)
@@ -18,5 +18,5 @@
                         rpy="0 0 0"/>
                 <geometry>
-                     <mesh filename="package://festo_phand_description/meshes/hand.STL"/>
+                     <mesh filename="package://festo_phand_description/meshes/hand_convex.STL"/>
                 </geometry>
             </collision>
@@ -42,5 +42,5 @@
                         rpy="0 0 0"/>
                 <geometry>
-                    <mesh filename="package://festo_phand_description/meshes/index_base_joint.STL"/>
+                    <mesh filename="package://festo_phand_description/meshes/index_base_joint_convex.STL"/>
                 </geometry>
             </collision>

File: festo_phand_description/urdf/thumb_macro.xacro (robot description, xacro)
@@ -23,5 +23,5 @@
                         rpy="0 0 0"/>
                 <geometry>
-                        <mesh filename="package://festo_phand_description/meshes/thumb/drive.STL"/>
+                        <mesh filename="package://festo_phand_description/meshes/thumb/drive_convex.STL"/>
                 </geometry>
             </collision>
@@ -47,5 +47,5 @@
                         rpy="0 0 0"/>
                 <geometry>
-                        <mesh filename="package://festo_phand_description/meshes/thumb/thumb_base.STL"/>
+                        <mesh filename="package://festo_phand_description/meshes/thumb/thumb_base_convex.STL"/>
                 </geometry>
             </collision>

File: festo_phand_description/urdf/wrist_macro.xacro (robot description, xacro)
@@ -32,5 +32,5 @@
                         rpy="0 0 0"/>
                 <geometry>
-                     <mesh filename="package://festo_phand_description/meshes/wrist/wrist_base.STL"/>
+                     <mesh filename="package://festo_phand_description/meshes/wrist/wrist_base_convex.STL"/>
                 </geometry>
             </collision>
@@ -43,5 +43,5 @@
                         rpy="0 0 0"/>
                 <geometry>
-                        <mesh filename="package://festo_phand_description/meshes/static_components.STL"/>
+                        <mesh filename="package://festo_phand_description/meshes/static_components_convex.STL"/>
                 </geometry>
                      <xacro:black />
@@ -52,5 +52,5 @@
                         rpy="0 0 0"/>
                 <geometry>
-                     <mesh filename="package://festo_phand_description/meshes/wrist/wrist_base.STL"/>
+                     <mesh filename="package://festo_phand_description/meshes/static_components_convex.STL"/>
                 </geometry>
             </collision>
@@ -72,5 +72,5 @@
                         rpy="0 0 0"/>
                 <geometry>
-                    <mesh filename="package://festo_phand_description/meshes/wrist/wrist_top.STL"/>
+                    <mesh filename="package://festo_phand_description/meshes/wrist/wrist_top_convex.STL"/>
                 </geometry>
             </collision>
